File: PCB/DesignESP32PCB.kicad_sch (KiCad schematic)
At the start: 26 parts, among them U1 ESP32-S3-MINI-1-N8, U2 ESD7104MUTAG, U3 TLV75801PDRV, U4 ENS210

Commit message: pcb
Parts:
- removed C5: 0.1uF, Capacitor_SMD:C_0603_1608Metric, symbol Device:C_Small
- removed D1: WS2812B, LED_SMD:LED_WS2812B_PLCC4_5.0x5.0mm_P3.2mm, symbol LED:WS2812B
- removed R4, R5: 10k, Resistor_SMD:R_0603_1608Metric, symbol Device:R_Small
- removed U4: ENS210, Package_DFN_QFN:AMS_QFN-4-1EP_2x2mm_P0.95mm_EP0.7x1.6mm, symbol Sensor_Humidity:ENS210
- added C10, C12, C13, C16, C18, C20, C8: 4.7uF, symbol Device:C
- added C11, C14, C15, C17, C19, C21, C9: 0.1uF, symbol Device:C
- added C22, C23: 0.1uF, Capacitor_SMD:C_1206_3216Metric_Pad1.33x1.80mm_HandSolder, symbol Device:C
- added C24, C25: 50uF, Capacitor_SMD:C_1206_3216Metric_Pad1.33x1.80mm_HandSolder, symbol Device:C
- added C26, C27, C30: 10uF, symbol Device:C
- added C28, C29, C31: 22uF, symbol Device:C
- added D3, D4, D5, D6, D7, D8, D9: SFH_4545, SFH_4545:DIO_SFH_4545, symbol SFH_4545:SFH_4545
- added J2: Left_Encoder, symbol Connector_Generic:Conn_01x06
- added J4: Right_Encoder, symbol Connector_Generic:Conn_01x06
- added J5: XT30PW-M, XT30PW-M:AMASS_XT30PW-M, symbol XT30PW-M:XT30PW-M
- added J6: Fan Motor, symbol Connector_Generic:Conn_01x02
- added L_MOTOR_DRIVER1, R_MOTOR_DRIVER1: DRV8871DDARQ1, DRV8871DDARQ1:DDA0008H_N_TEX, symbol DRV8871:DRV8871DDARQ1
- added Q1, Q15, Q2, Q3, Q4, Q5, Q6, Q7: NMOS, symbol Simulation_SPICE:NMOS
- added Q10, Q11, Q12, Q13, Q14, Q8, Q9: TEFT4300, TEFT4300:XDCR_TEFT4300, symbol TEFT4300:TEFT4300
- added R10, R12, R15, R16, R21, R24, R27, R37: 100Ω, symbol Device:R
- added R11, R13, R17, R18, R22, R25, R28, R38: 47kΩ, symbol Device:R
- added R14, R19, R20, R23, R26, R29, R9: 10Ω, symbol Device:R
- added R30, R31, R32, R33, R34, R35, R36: 470Ω, symbol Device:R
- added R_L_MTR1, R_R_MTR1: 18kΩ, Resistor_SMD:R_1206_3216Metric_Pad1.30x1.75mm_HandSolder, symbol Device:R
- added SW3: 1101M2S3CQE2, 1101M2S3CQE2:1101M2S3CQE2, symbol 1101M2S3CQE2:1101M2S3CQE2
- added U4: ICM-42688-P, ICM-42688-P:PQFN50P300X250X97-14N, symbol ICM-42688-P:ICM-42688-P
- added U5: AMS1117-3.3, Package_TO_SOT_SMD:SOT-223-3_TabPin2, symbol Regulator_Linear:AMS1117-3.3
- added U6, U7: AMS1117-5.0, Package_TO_SOT_SMD:SOT-223-3_TabPin2, symbol Regulator_Linear:AMS1117-5.0
Connections:
- net GPIO11 is gone; now on net Reciever_1: J1.13 (Pin_13), U1.15 (IO11)
- net GPIO2 is gone; now on net Reciever_2: J1.4 (Pin_4), U1.6 (IO2)
- net GPIO4 is gone; now on net Reciever_3: J1.6 (Pin_6), U1.8 (IO4)
- net GPIO5 is gone; now on net Reciever_4: J1.7 (Pin_7), U1.9 (IO5)
- net GPIO6 is gone; now on net Reciever_5: J1.8 (Pin_8), U1.10 (IO6)
- net GPIO7 is gone; now on net Reciever_6: J1.9 (Pin_9), U1.11 (IO7)
- net I2C_SCL is gone; now on net Reciever_7: J1.19 (Pin_19), U1.21 (IO17)
- net GND: now also C10.2, C11.2, C12.2, C13.2, C14.2, C15.2, C16.2, C17.2, C18.2, C19.2, C20.2, C21.2, C22.2, C23.2, C24.2, C25.2, C26.2, C27.2, C28.2, C29.2, C30.2, C31.2, C8.2, C9.2, J2.1 (Pin_1), J4.1 (Pin_1), J5.N, L_MOTOR_DRIVER1.1 (GND), L_MOTOR_DRIVER1.7 (PGND), L_MOTOR_DRIVER1.9 (PAD), Q1.3 (S), Q15.3 (S), Q2.3 (S), Q3.3 (S), Q4.3 (S), Q5.3 (S), Q6.3 (S), Q7.3 (S), R11.1, R13.1, R17.1, R18.1, R22.1, R25.1, R28.1, R30.1, R31.1, R32.1, R33.1, R34.1, R35.1, R36.1, R38.1, R_L_MTR1.2, R_MOTOR_DRIVER1.1 (GND), R_MOTOR_DRIVER1.7 (PGND), R_MOTOR_DRIVER1.9 (PAD), R_R_MTR1.2, U4.1 (AP_SDO/AP_AD0), U4.10 (RESV_10), U4.11 (RESV_11), U4.2 (RESV_2), U4.3 (RESV_3), U4.6 (GND), U4.7 (RESV_7), U4.9 (INT2/FSYNC/CLKIN), U5.1 (GND), U6.1 (GND), U7.1 (GND)
- net 3V3 renamed +3.3V
- net +3.3V: now also C28.1, J2.4 (Pin_4), J4.4 (Pin_4), Q10.C, Q11.C, Q12.C, Q13.C, Q14.C, Q8.C, Q9.C, U4.12 (AP_CS), U4.5 (VDDIO), U4.8 (VDD), U5.2 (VO)
- net GPIO1 renamed Reciever_1
- net Reciever_1: now also Q8.E, R30.2
- net GPIO12 renamed Reciever_2
- net Reciever_2: now also Q9.E, R31.2
- net GPIO13 renamed Reciever_3
- net Reciever_3: now also Q10.E, R32.2
- net GPIO14 renamed Reciever_4
- net Reciever_4: now also Q11.E, R33.2
- net GPIO15 renamed Reciever_5
- net Reciever_5: now also Q12.E, R34.2
- net GPIO16 renamed Reciever_6
- net Reciever_6: now also Q13.E, R35.2
- net GPIO21 renamed FAN_PWM
- net FAN_PWM: now also R37.1
- net GPIO35 renamed L_IN1
- net L_IN1: now also L_MOTOR_DRIVER1.3 (IN1)
- net GPIO36 renamed L_IN2
- net L_IN2: now also L_MOTOR_DRIVER1.2 (IN2)
- net GPIO37 renamed R_IN1
- net R_IN1: now also R_MOTOR_DRIVER1.3 (IN1)
- net GPIO38 renamed R_IN2
- net R_IN2: now also R_MOTOR_DRIVER1.2 (IN2)
- net GPIO39 renamed L_A
- net L_A: now also J2.3 (Pin_3)
- net GPIO40 renamed L_B
- net L_B: now also J2.2 (Pin_2)
- net GPIO41 renamed R_A
- net R_A: now also J4.3 (Pin_3)
- net GPIO42 renamed R_B
- net R_B: now also J4.2 (Pin_2)
- net GPIO47 renamed IMU_SDA
- net IMU_SDA: now also U4.14 (AP_SDA/AP_SDIO/AP_SDI)
- net GPIO48 renamed IMU_SCL
- net IMU_SCL: now also U4.13 (AP_SCL/AP_SCLK)
- net GPIO8 renamed Reciever_7
- net Reciever_7: now also Q14.E, R36.2
- net I2C_SDA renamed IMU_INT
- net IMU_INT: now also U4.4 (INT1/INT)
- new net: D6.A, R20.2
- new net: D6.C, Q4.1 (D)
- new net: D4.C, Q2.1 (D)
- new net: Q2.2 (G), R12.2, R13.2
- new net: Q7.2 (G), R27.2, R28.2
- new net: D8.C, Q6.1 (D)
- new net: Q6.2 (G), R24.2, R25.2
- new net: D8.A, R26.2
- new net: R_MOTOR_DRIVER1.4 (ILIM), R_R_MTR1.1
- new net: J4.6 (Pin_6), R_MOTOR_DRIVER1.6 (OUT1)
- new net: J4.5 (Pin_5), R_MOTOR_DRIVER1.8 (OUT2)
- new net: Q4.2 (G), R16.2, R18.2
- new net: Q1.2 (G), R10.2, R11.2
- new net: D3.A, R9.2
- new net: D7.C, Q5.1 (D)
- new net: Q5.2 (G), R21.2, R22.2
- new net: D9.C, Q7.1 (D)
- new net: Q15.2 (G), R37.2, R38.2
- new net: D5.A, R19.2
- new net: D3.C, Q1.1 (D)
- new net: C31.1, J6.2 (Pin_2), U7.2 (VO)
- new net: J6.1 (Pin_1), Q15.1 (D)
- new net: J5.P, SW3.1
- new net: D5.C, Q3.1 (D)
- new net: L_MOTOR_DRIVER1.4 (ILIM), R_L_MTR1.1
- new net: J2.6 (Pin_6), L_MOTOR_DRIVER1.6 (OUT1)
- new net: J2.5 (Pin_5), L_MOTOR_DRIVER1.8 (OUT2)
- new net: D7.A, R23.2
- new net: Q3.2 (G), R15.2, R17.2
- new net: D9.A, R29.2
- new net: D4.A, R14.2
- new net +5V: C10.1, C11.1, C12.1, C13.1, C14.1, C15.1, C16.1, C17.1, C18.1, C19.1, C20.1, C21.1, C29.1, C8.1, C9.1, R14.1, R19.1, R20.1, R23.1, R26.1, R29.1, R9.1, U6.2 (VO)
- new net +8V: C22.1, C23.1, C24.1, C25.1, C26.1, C27.1, C30.1, L_MOTOR_DRIVER1.5 (VM), R_MOTOR_DRIVER1.5 (VM), SW3.2, U5.3 (VI), U6.3 (VI), U7.3 (VI)
- new net Emitter_1: R10.1
- new net Emitter_2: R12.1
- new net Emitter_3: R21.1
- new net Emitter_4: R27.1
- new net Emitter_5: R15.1
- new net Emitter_6: R16.1
- new net Emitter_7: R24.1
Other:
- note added: "Emitters"
- note added: "Fan Motor"
- note added: "Motor Drivers"
- note added: "Power Dist"
- note added: "Recievers"
- note added: "https://jlcpcb.com/partdetail/TDKInvenSense-ICM_42688P/C1850418"
- moved on the sheet: C1, C2, C6, C7, D2, J1, J3, R6, R7, R8, U1, U3
